Commit message: added world camera to articulation

File: movit_ws/src/panda_description/urdf/Franka.urdf (robot description, URDF)
Before this commit: robot Franka, 17 links, 16 joints
Links:
- link Franka_panda_hand: geometry collision mesh filename=meshes/Franka_panda_hand_geometry_panda_hand.obj scale=1. 1. 1.; visual mesh filename=meshes/Franka_panda_hand_geometry_panda_hand.obj scale=1. 1. 1.
- link Franka_panda_leftfinger: mass 0.014 -> 0.0140552; geometry collision mesh filename=meshes/Franka_panda_leftfinger_geometry_panda_leftfinger.obj scale=1. 1. 1.; visual mesh filename=meshes/Franka_panda_leftfinger_geometry_panda_leftfinger.obj scale=1. 1. 1.
- link Franka_panda_link1: geometry collision mesh filename=meshes/Franka_panda_link1_geometry_panda_link1.obj scale=1. 1. 1.; visual mesh filename=meshes/Franka_panda_link1_geometry_panda_link1.obj scale=1. 1. 1.
- link Franka_panda_link2: geometry collision mesh filename=meshes/Franka_panda_link2_geometry_panda_link2.obj scale=1. 1. 1.; visual mesh filename=meshes/Franka_panda_link2_geometry_panda_link2.obj scale=1. 1. 1.
- link Franka_panda_link3: geometry collision mesh filename=meshes/Franka_panda_link3_geometry_panda_link3.obj scale=1. 1. 1.; visual mesh filename=meshes/Franka_panda_link3_geometry_panda_link3.obj scale=1. 1. 1.
- link Franka_panda_link4: geometry collision mesh filename=meshes/Franka_panda_link4_geometry_panda_link4.obj scale=1. 1. 1.; visual mesh filename=meshes/Franka_panda_link4_geometry_panda_link4.obj scale=1. 1. 1.
- link Franka_panda_link5: geometry collision mesh filename=meshes/Franka_panda_link5_geometry_panda_link5.obj scale=1. 1. 1.; visual mesh filename=meshes/Franka_panda_link5_geometry_panda_link5.obj scale=1. 1. 1.
- link Franka_panda_link6: geometry collision mesh filename=meshes/Franka_panda_link6_geometry_panda_link6.obj scale=1. 1. 1.; visual mesh filename=meshes/Franka_panda_link6_geometry_panda_link6.obj scale=1. 1. 1.
- link Franka_panda_link7: geometry collision mesh filename=meshes/Franka_panda_link7_geometry_panda_link7.obj scale=1. 1. 1.; visual mesh filename=meshes/Franka_panda_link7_geometry_panda_link7.obj scale=1. 1. 1.
- link Franka_panda_rightfinger: mass 0.014 -> 0.0140552; geometry collision mesh filename=meshes/Franka_panda_rightfinger_geometry_panda_rightfinger.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 scale=1. 1. 1.; visual mesh filename=meshes/Franka_panda_rightfinger_geometry_panda_rightfinger.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 scale=1. 1. 1.
- link Gemini2_hand: geometry visual mesh filename=meshes/Orbbec_Gemini2_back_cover_back_cover.obj scale=1. 1. 1.; visual mesh filename=meshes/Orbbec_Gemini2_camera_ldm_camera_ldm.obj scale=1. 1. 1.
- link Root: geometry collision mesh filename=meshes/Franka_panda_link0_geometry_panda_link0.obj scale=1. 1. 1.; visual mesh filename=meshes/Franka_panda_link0_geometry_panda_link0.obj scale=1. 1. 1.
Joints:
- joint PandaHandJoint: origin xyz=0.0449043 -0.0000857 0.046555  rpy=0 0 -1.553343 -> xyz=0.0449043 -0.0000857 0.046555  rpy=0. 0. -1.553343
- joint joint_Gemini2_hand-Stream_ir_right: origin xyz=0.025 -0.0000001 0.0061398 rpy=3.1415927 0 -3.1415927 -> xyz=0.025 -0.0000001 0.0061398 rpy=3.1415927 0. -3.1415927
- joint joint_Gemini2_hand-Stream_rgb: origin xyz=0.010989 -0.0000076 0.0076121 rpy=3.1415927 0 -3.1415927 -> xyz=0.010989 -0.0000076 0.0076121 rpy=3.1415927 0. -3.1415927
- joint joint_Gemini2_hand-gemini_hand_depth: origin xyz=-0.025 -0 0.0061398 rpy=3.1415927 0 -3.1415927 -> xyz=-0.025 -0. 0.0061398 rpy=3.1415927 0. -3.1415927
- joint joint_Gemini2_hand-gemini_hand_rgb: origin xyz=-0.025 -0 0.0061398 rpy=3.1415927 0 -3.1415927 -> xyz=-0.025 -0. 0.0061398 rpy=3.1415927 0. -3.1415927
- joint panda_finger_joint1: axis 1. 0 0 -> 1. 0. 0.; limit lower=0 upper=0.04 effort=7.1999998 velocity=10. -> lower=0. upper=0.04 effort=7.1999998 velocity=10.; origin xyz=0 -0 0.0584 rpy=0 -0 1.5707963 -> xyz=0. -0. 0.0584 rpy=0. -0. 1.5707963
- joint panda_finger_joint2: axis 1. 0 0 -> 1. 0. 0.; limit lower=0 upper=0.04 effort=0 velocity=10. -> lower=0. upper=0.04 effort=0. velocity=10.; origin xyz=0 -0 0.0584 rpy=-0 0 -1.5707964 -> xyz=0. -0. 0.0584 rpy=-0. 0. -1.5707964
- joint panda_hand_joint: origin xyz=-0.0000001 -0.0000001 0  rpy=1.5707964 -0.7853981 -1.5707964 -> xyz=-0.0000001 -0.0000001 0.  rpy=1.5707964 -0.7853981 -1.5707964
- joint panda_joint1: axis 1. 0 0 -> 1. 0. 0.; origin xyz=-0 0 0.333 rpy=0 -1.5707963 0  -> xyz=-0. 0. 0.333 rpy=0. -1.5707963 0. 
- joint panda_joint2: axis 1. 0 0 -> 1. 0. 0.; origin xyz=0.0000003 0.0000001 -0  rpy=0 0 1.5707964 -> xyz=0.0000003 0.0000001 -0.  rpy=0. 0. 1.5707964
- joint panda_joint3: axis 1. 0 0 -> 1. 0. 0.; origin xyz=-0.0000001 -0.3159997 0  rpy=-0.0000002 -0.0000002 -1.5707958 -> xyz=-0.0000001 -0.3159997 0.  rpy=-0.0000002 -0.0000002 -1.5707958
- joint panda_joint4: axis 1. 0 0 -> 1. 0. 0.; origin xyz=-0 -0.0000001 -0.0824999 rpy=-0.0000002 0.0000002 -1.5707968 -> xyz=-0. -0.0000001 -0.0824999 rpy=-0.0000002 0.0000002 -1.5707968
- joint panda_joint5: axis 1. 0 0 -> 1. 0. 0.
- joint panda_joint6: axis 1. 0 0 -> 1. 0. 0.
- joint panda_joint7: axis 1. 0 0 -> 1. 0. 0.; origin xyz=-0.0000002 -0.0000005 -0.0879998 rpy=-0 0 -1.5707996 -> xyz=-0.0000002 -0.0000005 -0.0879998 rpy=-0. 0. -1.5707996
- joint panda_joint8: origin xyz=0.1069999 0.0000004 -0.0000002 rpy=3.1415925 0 -3.1415894 -> xyz=0.1069999 0.0000004 -0.0000002 rpy=3.1415925 0. -3.1415894

Commit message: streaming depth and rgb properly now

File: movit_ws/src/panda_description/urdf/Franka.urdf (robot description, URDF)
Before this commit: robot Franka, 17 links, 16 joints
Links:
- removed link Stream_ir_right
- removed link Stream_rgb
- removed link gemini_hand_depth
- removed link gemini_hand_rgb
- added link Gemini2_hand_Orbbec_Gemini2_camera_ir_left_camera_left_gemini_hand_depth
- added link Gemini2_hand_Orbbec_Gemini2_camera_ir_left_camera_left_gemini_hand_rgb
- added link Gemini2_hand_Orbbec_Gemini2_camera_ir_right_camera_right_Stream_ir_right
- added link Gemini2_hand_Orbbec_Gemini2_camera_rgb_camera_rgb_Stream_rgb
- added link Gemini2_world; visual mesh filename=package://panda_description/meshes/Gemini2_world_Orbbec_Gem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 scale=1. 1. 1.; visual mesh filename=package://panda_description/meshes/Gemini2_world_Orbbec_Gem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 scale=1. 1. 1.
- added link Gemini2_world_Orbbec_Gemini2_camera_ir_left_camera_left_Stream_depth
- added link Gemini2_world_Orbbec_Gemini2_camera_ir_left_camera_left_Stream_ir_left
- added link Gemini2_world_Orbbec_Gemini2_camera_ir_right_camera_right_Stream_ir_right
- added link Gemini2_world_Orbbec_Gemini2_camera_rgb_camera_rgb_Stream_rgb
- link Franka_panda_hand: geometry collision mesh filename=package://panda_description/meshes/Franka_panda_hand_geomet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 scale=1. 1. 1.; visual mesh filename=package://panda_description/meshes/Franka_panda_hand_geomet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 scale=1. 1. 1.
- link Franka_panda_leftfinger: mass 0.0140552 -> 0.014; geometry collision mesh filename=package://panda_description/meshes/Franka_panda_leftfinger_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 scale=1. 1. 1.; visual mesh filename=package://panda_description/meshes/Franka_panda_leftfinger_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 scale=1. 1. 1.
- link Franka_panda_link1: geometry collision mesh filename=package://panda_description/meshes/Franka_panda_link1_geome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 scale=1. 1. 1.; visual mesh filename=package://panda_description/meshes/Franka_panda_link1_geome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 scale=1. 1. 1.
- link Franka_panda_link2: geometry collision mesh filename=package://panda_description/meshes/Franka_panda_link2_geome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 scale=1. 1. 1.; visual mesh filename=package://panda_description/meshes/Franka_panda_link2_geome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 scale=1. 1. 1.
- link Franka_panda_link3: geometry collision mesh filename=package://panda_description/meshes/Franka_panda_link3_geome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 scale=1. 1. 1.; visual mesh filename=package://panda_description/meshes/Franka_panda_link3_geome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 scale=1. 1. 1.
- link Franka_panda_link4: geometry collision mesh filename=package://panda_description/meshes/Franka_panda_link4_geome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 scale=1. 1. 1.; visual mesh filename=package://panda_description/meshes/Franka_panda_link4_geome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 scale=1. 1. 1.
- link Franka_panda_link5: geometry collision mesh filename=package://panda_description/meshes/Franka_panda_link5_geome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 scale=1. 1. 1.; visual mesh filename=package://panda_description/meshes/Franka_panda_link5_geome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 scale=1. 1. 1.
- link Franka_panda_link6: geometry collision mesh filename=package://panda_description/meshes/Franka_panda_link6_geome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 scale=1. 1. 1.; visual mesh filename=package://panda_description/meshes/Franka_panda_link6_geome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 scale=1. 1. 1.
- link Franka_panda_link7: geometry collision mesh filename=package://panda_description/meshes/Franka_panda_link7_geome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 scale=1. 1. 1.; visual mesh filename=package://panda_description/meshes/Franka_panda_link7_geome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 scale=1. 1. 1.
- link Franka_panda_rightfinger: mass 0.0140552 -> 0.014; geometry collision mesh filename=package://panda_description/meshes/Franka_panda_rightfinger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 scale=1. 1. 1.; visual mesh filename=package://panda_description/meshes/Franka_panda_rightfinger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 scale=1. 1. 1.
- link Gemini2_hand: geometry visual mesh filename=package://panda_description/meshes/Gemini2_hand_Orbbec_Gemi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 scale=1. 1. 1.; visual mesh filename=package://panda_description/meshes/Gemini2_hand_Orbbec_Gemi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 scale=1. 1. 1.
- link Root: geometry collision mesh filename=package://panda_description/meshes/Franka_panda_link0_geome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 scale=1. 1. 1.; visual mesh filename=package://panda_description/meshes/Franka_panda_link0_geome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 scale=1. 1. 1.
Joints:
- removed joint joint_Gemini2_hand-Stream_ir_right
- removed joint joint_Gemini2_hand-Stream_rgb
- removed joint joint_Gemini2_hand-gemini_hand_depth
- removed joint joint_Gemini2_hand-gemini_hand_rgb
- added joint joint_Gemini2_hand-Gemini2_hand_Orbbec_Gemini2_camera_ir_left_camera_left_gemini_hand_depth: type fixed, parent Gemini2_hand, child Gemini2_hand_Orbbec_Gemini2_camera_ir_left_camera_left_gemini_hand_depth, origin xyz=-0.025 -0. 0.0061398 rpy=3.1415927 0. -3.1415927
- added joint joint_Gemini2_hand-Gemini2_hand_Orbbec_Gemini2_camera_ir_left_camera_left_gemini_hand_rgb: type fixed, parent Gemini2_hand, child Gemini2_hand_Orbbec_Gemini2_camera_ir_left_camera_left_gemini_hand_rgb, origin xyz=-0.025 -0. 0.0061398 rpy=3.1415927 0. -3.1415927
- added joint joint_Gemini2_hand-Gemini2_hand_Orbbec_Gemini2_camera_ir_right_camera_right_Stream_ir_right: type fixed, parent Gemini2_hand, child Gemini2_hand_Orbbec_Gemini2_camera_ir_right_camera_right_Stream_ir_right, origin xyz=0.025 -0.0000001 0.0061398 rpy=3.1415927 0. -3.1415927
- added joint joint_Gemini2_hand-Gemini2_hand_Orbbec_Gemini2_camera_rgb_camera_rgb_Stream_rgb: type fixed, parent Gemini2_hand, child Gemini2_hand_Orbbec_Gemini2_camera_rgb_camera_rgb_Stream_rgb, origin xyz=0.010989 -0.0000076 0.0076121 rpy=3.1415927 0. -3.1415927
- added joint joint_Gemini2_world-Gemini2_world_Orbbec_Gemini2_camera_ir_left_camera_left_Stream_depth: type fixed, parent Gemini2_world, child Gemini2_world_Orbbec_Gemini2_camera_ir_left_camera_left_Stream_depth, origin xyz=-0.025 0. 0.0061398 rpy=-3.1415927 0. -3.1415927
- added joint joint_Gemini2_world-Gemini2_world_Orbbec_Gemini2_camera_ir_left_camera_left_Stream_ir_left: type fixed, parent Gemini2_world, child Gemini2_world_Orbbec_Gemini2_camera_ir_left_camera_left_Stream_ir_left, origin xyz=-0.025 0. 0.0061398 rpy=-3.1415927 0. 3.1415927
- added joint joint_Gemini2_world-Gemini2_world_Orbbec_Gemini2_camera_ir_right_camera_right_Stream_ir_right: type fixed, parent Gemini2_world, child Gemini2_world_Orbbec_Gemini2_camera_ir_right_camera_right_Stream_ir_right, origin xyz=0.025 -0.0000001 0.0061398 rpy=-3.1415927 0. -3.1415927
- added joint joint_Gemini2_world-Gemini2_world_Orbbec_Gemini2_camera_rgb_camera_rgb_Stream_rgb: type fixed, parent Gemini2_world, child Gemini2_world_Orbbec_Gemini2_camera_rgb_camera_rgb_Stream_rgb, origin xyz=0.010989 -0.0000076 0.0076121 rpy=-3.1415927 0. -3.1415927
- added joint world_camera_joint: type fixed, parent Root, child Gemini2_world, origin xyz=0.3212462 0. 1.3169613 rpy=3.1415927 0. -1.5707964
